Commit message: Implement all 15 bug fixes from critical review

File: assets/zero_g_servicer.urdf (robot description, URDF)
Before this commit: robot zero_g_servicer, 10 links, 9 joints
Joints:
- joint gripper_joint_right: axis (none) -> 0 -1 0; limit (none) -> lower=0.0 upper=0.03 effort=10.0 velocity=0.5; type fixed -> prismatic

Commit message: Fix all critical issues identified in RL audit report

File: assets/zero_g_servicer.urdf (robot description, URDF)
Before this commit: robot zero_g_servicer, 10 links, 9 joints
Links:
- link shoulder_link_2: geometry collision cylinder length=0.2 radius=0.04; visual cylinder length=0.2 radius=0.04
- link shoulder_link_3: geometry collision cylinder length=0.1 radius=0.04; visual cylinder length=0.1 radius=0.04
- link wrist_link_0: geometry collision cylinder length=0.05 radius=0.03; visual cylinder length=0.05 radius=0.03
- link wrist_link_1: geometry collision box size=0.08 0.04 0.04; visual box size=0.08 0.04 0.04
